Commit message: fixed urdf and sim

File: ros2_ws/src/maurice_bot/maurice_sim/urdf/maurice.urdf (robot description, URDF)
Before this commit: robot maurice_bot, 9 links, 8 joints
Links:
- removed link world
- added link base_root, mass 0.01
- added link base_x, mass 0.01
- added link base_y, mass 0.01
Joints:
- removed joint arm_camera_joint
- removed joint base_joint
- added joint base_x: type prismatic, parent base_root, child base_x, origin xyz=0 0 0 rpy=0 0 0, axis 1 0 0, limit lower=0 upper=0 effort=0 velocity=0
- added joint base_y: type prismatic, parent base_x, child base_y, origin xyz=0 0 0 rpy=0 0 0, axis 0 1 0, limit lower=0 upper=0 effort=0 velocity=0
- added joint base_yaw: type revolute, parent base_y, child base_link, origin xyz=0 0 0 rpy=0 0 0, axis 0 0 1, limit lower=-3.1416 upper=3.1416 effort=0.0 velocity=0.0
- added joint fixed_arm_camera_link: type fixed, parent link5, child arm_camera_link, origin xyz=0.00454 0 0.05448 rpy=0 0 0
- joint joint1: limit lower=-3.14 upper=3.14 effort=1.5 velocity=1.0 -> lower=-3.1416 upper=3.1416 effort=0.0 velocity=0.0
- joint joint2: limit lower=-3.14 upper=3.14 effort=1.5 velocity=1.0 -> lower=-3.1416 upper=3.1416 effort=0.0 velocity=0.0
- joint joint3: limit lower=-3.14 upper=3.14 effort=1.5 velocity=1.0 -> lower=-3.1416 upper=3.1416 effort=0.0 velocity=0.0
- joint joint4: limit lower=-3.14 upper=3.14 effort=0.6 velocity=1.0 -> lower=-3.1416 upper=3.1416 effort=0.0 velocity=0.0
- joint joint5: limit lower=-3.14 upper=3.14 effort=0.6 velocity=1.0 -> lower=-3.1416 upper=3.1416 effort=0.0 velocity=0.0
- joint joint6: axis 0 0 1 -> 0 0 -1; limit lower=-3.14 upper=3.14 effort=0.6 velocity=1.0 -> lower=-3.1416 upper=3.1416 effort=0.0 velocity=0.0; origin xyz=0.059 -0.0055 0 rpy=0 0 0 -> xyz=0.014 -0.0075 0 rpy=0 0 0

Commit message: Squash: new_arm_dev changes on top of main

File: ros2_ws/src/maurice_bot/maurice_sim/urdf/maurice.urdf (robot description, URDF)
Before this commit: robot maurice_bot, 11 links, 10 joints
Links:
- added link ee_link, mass 0.001; visual sphere radius=0.005
Joints:
- added joint ee_joint: type fixed, parent link5, child ee_link, origin xyz=0.09285 0 0 rpy=0 0 0
- joint joint1: origin xyz=0.0845 -0.0597 0.0583 rpy=0 0 0 -> xyz=0.086 -0.05285 0.04025 rpy=0 0 0
- joint joint2: origin xyz=0 0 0.01825 rpy=0 0 0 -> xyz=0 0 0.04225 rpy=0 0 0
- joint joint3: origin xyz=0.034 0 0.11825 rpy=0 0 0 -> xyz=0.02825 0 0.12125 rpy=0 0 0
- joint joint4: origin xyz=0.13609 0 0.00025 rpy=0 0 0 -> xyz=0.1375 0 -0.0045 rpy=0 0 0
- joint joint5: origin xyz=0.045 0.002 0 rpy=0 0 0 -> xyz=0.019 0 0 rpy=0 0 0
- joint joint6: axis 0 0 -1 -> 0 0 1; origin xyz=0.014 -0.0075 0 rpy=0 0 0 -> xyz=0.044 0.0091 0 rpy=0 0 0

Commit message: urdf updated

File: ros2_ws/src/maurice_bot/maurice_sim/urdf/maurice.urdf (robot description, URDF)
Before this commit: robot maurice_bot, 12 links, 11 joints
Links:
- removed link link6
- added link link61, mass 0.012; collision mesh filename=package://maurice_sim/meshes/link61.STL scale=0.001 0.001 0.001; visual mesh filename=package://maurice_sim/meshes/link61.STL scale=0.001 0.001 0.001
- added link link62, mass 0.012; collision mesh filename=package://maurice_sim/meshes/link62.STL scale=0.001 0.001 0.001; visual mesh filename=package://maurice_sim/meshes/link62.STL scale=0.001 0.001 0.001
- link link5: geometry collision mesh filename=package://maurice_sim/meshes/link5.STL scale=0.001 0.001 0.001; visual mesh filename=package://maurice_sim/meshes/link5.STL scale=0.001 0.001 0.001
Joints:
- removed joint joint6
- added joint joint61: type revolute, parent link5, child link61, origin xyz=0.044 -0.0091 0 rpy=0 0 0, axis 0 0 1, limit lower=-1.57 upper=1.57 effort=2.0 velocity=2.0
- added joint joint62: type revolute, parent link5, child link62, origin xyz=0.044 0.0091 0 rpy=0 0 0, axis 0 0 1, limit lower=-1.57 upper=1.57 effort=2.0 velocity=2.0, mimic joint=joint61 multiplier=-1 offset=0

Commit message: urdf with both fingers

File: ros2_ws/src/maurice_bot/maurice_sim/urdf/maurice.urdf (robot description, URDF)
Before this commit: robot maurice_bot, 13 links, 12 joints
Joints:
- removed joint joint61
- removed joint joint62
- added joint joint6: type revolute, parent link5, child link61, origin xyz=0.044 -0.0091 0 rpy=0 0 0, axis 0 0 1, limit lower=-1.57 upper=1.57 effort=2.0 velocity=2.0
- added joint joint6M: type revolute, parent link5, child link62, origin xyz=0.044 0.0091 0 rpy=0 0 0, axis 0 0 1, limit lower=-1.57 upper=1.57 effort=2.0 velocity=2.0, mimic joint=joint6 multiplier=-1 offset=0

Commit message: link2 correct

File: ros2_ws/src/maurice_bot/maurice_sim/urdf/maurice.urdf (robot description, URDF)
Before this commit: robot maurice_bot, 13 links, 12 joints
Links:
- link link2: geometry collision cylinder length=0.1385 radius=0.025; visual mesh filename=package://maurice_sim/meshes/link2.STL scale=1 1 1

Commit message: link 3 correct

File: ros2_ws/src/maurice_bot/maurice_sim/urdf/maurice.urdf (robot description, URDF)
Before this commit: robot maurice_bot, 13 links, 12 joints
Links:
- link link3: geometry collision cylinder length=0.118 radius=0.023; visual mesh filename=package://maurice_sim/meshes/link3.STL scale=1 1 1
- link link61: geometry collision box size=0.048 0.016 0.0389; visual mesh filename=package://maurice_sim/meshes/link61.STL scale=0.001 0.001 0.001
- link link62: geometry collision box size=0.048 0.016 0.0389; visual mesh filename=package://maurice_sim/meshes/link62.STL scale=0.001 0.001 0.001

Commit message: optimized link 3 and fixed igners

File: ros2_ws/src/maurice_bot/maurice_sim/urdf/maurice.urdf (robot description, URDF)
Before this commit: robot maurice_bot, 13 links, 12 joints
Links:
- link link2: geometry collision box size=0.020 0.054 0.1385; visual mesh filename=package://maurice_sim/meshes/link2.STL scale=1 1 1

Commit message: some move it config stuff

File: ros2_ws/src/maurice_bot/maurice_sim/urdf/maurice.urdf (robot description, URDF)
Before this commit: robot maurice_bot, 13 links, 12 joints
Joints:
- joint joint1: limit lower=-3.1416 upper=3.1416 effort=0.0 velocity=0.0 -> lower=-1.5708 upper=1.5708 effort=2.0 velocity=2.0
- joint joint2: limit lower=-3.1416 upper=3.1416 effort=0.0 velocity=0.0 -> lower=-1.5708 upper=1.22 effort=2.0 velocity=2.0
- joint joint3: limit lower=-3.1416 upper=3.1416 effort=0.0 velocity=0.0 -> lower=-1.5708 upper=1.7453 effort=2.0 velocity=2.0
- joint joint4: limit lower=-3.1416 upper=3.1416 effort=0.0 velocity=0.0 -> lower=-1.9199 upper=1.7453 effort=2.0 velocity=2.0
- joint joint5: limit lower=-3.1416 upper=3.1416 effort=0.0 velocity=0.0 -> lower=-1.5708 upper=1.5708 effort=2.0 velocity=2.0
- joint joint6: limit lower=-1.57 upper=1.57 effort=2.0 velocity=2.0 -> lower=-0.8727 upper=0.3491 effort=2.0 velocity=2.0
- joint joint6M: limit lower=-1.57 upper=1.57 effort=2.0 velocity=2.0 -> lower=-0.8727 upper=0.3491 effort=2.0 velocity=2.0

Commit message: Updated rpy and scale
Fixed rpy visual offset and scale to 0 and 1 to accurately simulate robot with meshes

File: ros2_ws/src/maurice_bot/maurice_sim/urdf/maurice.urdf (robot description, URDF)
Before this commit: robot maurice_bot, 16 links, 15 joints
Links:
- link link5: geometry collision mesh filename=package://maurice_sim/meshes/link5.STL scale=1 1 1; visual mesh filename=package://maurice_sim/meshes/link5.STL scale=1 1 1
- link link61: geometry collision box size=0.048 0.016 0.0389; visual mesh filename=package://maurice_sim/meshes/link61.STL scale=1 1 1
- link link62: geometry collision box size=0.048 0.016 0.0389; visual mesh filename=package://maurice_sim/meshes/link62.STL scale=1 1 1
Joints:
- joint joint_head: axis (none) -> 0 1 0; limit (none) -> lower=-0.1745 upper=0.5236 effort=2.0 velocity=2.0; type fixed -> revolute

Commit message: Deleting redundant urdf components

File: ros2_ws/src/maurice_bot/maurice_sim/urdf/maurice.urdf (robot description, URDF)
Before this commit: robot maurice_bot, 16 links, 15 joints
Links:
- removed link base_root
- removed link base_x
- removed link base_y
Joints:
- removed joint base_x
- removed joint base_y
- removed joint base_yaw
